Commit message: Robo feito

File: src/rm_description/urdf/properties.xacro (robot description, xacro)
@@ -6,19 +6,8 @@
   <!-- ============================================ -->
   <!-- Propriedades da Base -->
-  <xacro:property name="base_radius" value="0.1"/>
-  <xacro:property name="base_height" value="0.05"/>
+  <xacro:property name="base_height" value="0.1"/>
   <xacro:property name="base_mass" value="2.0"/>
-  <!-- TAREFA: Defina as propriedades do Link 1 -->
-  <!-- Use os valores da tabela de referência (seção 2.2) -->
-  <xacro:property name="link1_length" value="0.3"/>
-  <xacro:property name="link1_radius" value="0.03"/>
-  <xacro:property name="link1_mass" value="1.0"/>
-  <!-- TAREFA: Defina as propriedades do Link 2 -->
-  <xacro:property name="link2_length" value="0.25"/>
-  <xacro:property name="link2_radius" value="0.025"/>
-  <xacro:property name="link2_mass" value="0.8"/>
-  <!-- Propriedades do End Effector -->
-  <xacro:property name="ee_radius" value="0.02"/>
-  <xacro:property name="ee_mass" value="0.1"/>
+  <xacro:property name="base_length" value="0.5"/>
+  <xacro:property name="base_width" value="0.3"/>
   <!-- ============================================ -->
   <!-- MATERIAIS (cores)                            -->
