Commit message: Robo dentro da casa (Sem sensores)

File: src/rm_description/urdf/differential_robot.xacro (robot description, xacro)
@@ -18,5 +18,19 @@
   <!-- ==================== -->
   <link name="base_footprint">
+    <inertial>
+      <origin xyz="0 0 0"/>
+      <mass value="1.0"/>
+      <inertia
+        ixx="0.1"
+        ixy="0.0"
+        ixz="0.0"
+        iyy="0.1"
+        iyz="0.0"
+        izz="0.1"/>
+    </inertial>
   </link>
+  <gazebo reference="base_footprint">
+    <gravity>false</gravity>
+  </gazebo>
   <!-- ==================== -->
   <!-- BASE LINK            -->
@@ -55,7 +69,4 @@
   <xacro:wheels
   name="left_wheel"
-  length="0.05"
-  radius="0.15"
-  mass="0.5"
   material="blue"/>
   <joint name="left_wheel_joint" type="continuous">
@@ -64,12 +75,9 @@
   <origin xyz="0 ${base_width/2 + 0.05/2} 0"
           rpy="1.5708 0 0"/>
-  <axis xyz="0 0 11"/>
+  <axis xyz="0 0 1"/>
   </joint>
   <!-- Roda Direita -->
   <xacro:wheels
   name="right_wheel"
-  length="0.05"
-  radius="0.15"
-  mass="0.5"
   material="blue"/>
   <joint name="right_wheel_joint" type="continuous">
@@ -82,5 +90,5 @@
   name="caster_ball"
   radius="0.1"
-  mass="0.5"
+  mass="0.7"
   material="red"/>
   <joint name="caster_joint" type="fixed">

File: src/rm_description/urdf/robot.urdf (robot description, URDF)
Before this commit: robot differential_robot, 3 links, 2 joints
Links:
- added link caster_ball, mass 0.5; collision sphere radius=0.1; visual sphere radius=0.1
- added link right_wheel, mass 0.5; collision cylinder length=0.05 radius=0.15; visual cylinder length=0.05 radius=0.15
- link left_wheel: geometry collision cylinder length=0.05 radius=0.15; visual cylinder length=0.05 radius=0.15
Joints:
- added joint caster_joint: type fixed, parent base_link, child caster_ball, origin xyz=0.25 0 -0.05 rpy=0 0 0
- added joint right_wheel_joint: type continuous, parent base_link, child right_wheel, origin xyz=0 -0.175 0 rpy=1.5708 0 0, axis 0 0 1
- joint base_joint: origin xyz=0 0 0.05 rpy=0 0 0 -> xyz=0 0 0.15000000000000002 rpy=0 0 0
- joint left_wheel_joint: axis 0 1 0 -> 0 0 1; origin xyz=0 0.15 0 rpy=0 1.5707 0 -> xyz=0 0.175 0 rpy=1.5708 0 0

File: src/rm_description/urdf/wheels.xacro (robot description, xacro)
@@ -5,4 +5,7 @@
   <!-- Contém componentes reutilizáveis             -->
   <!-- ============================================ -->
+  <xacro:property name="wheel_radius" value="0.15"/>
+  <xacro:property name="wheel_length" value="0.05"/>
+  <xacro:property name="wheel_mass" value="0.5"/>
   <!-- ==================== -->
   <!-- MACRO: LINK CILÍNDRICO -->
@@ -18,5 +21,5 @@
       - material: nome do material (definido em properties.xacro)
   -->
-  <xacro:macro name="wheels" params="name length radius mass material">
+  <xacro:macro name="wheels" params="name material">
     <link name="${name}">
       <visual>
@@ -24,5 +27,5 @@
         <origin xyz="0 0 0" rpy="0 0 0"/>
         <geometry>
-          <cylinder radius="${radius}" length="${length}"/>
+          <cylinder radius="${wheel_radius}" length="${wheel_length}"/>
         </geometry>
         <material name="${material}"/>
@@ -31,17 +34,17 @@
         <origin xyz="0 0 0" rpy="0 0 0"/>
         <geometry>
-          <cylinder radius="${radius}" length="${length}"/>
+          <cylinder radius="${wheel_radius}" length="${wheel_length}"/>
         </geometry>
       </collision>
       <inertial>
         <origin xyz="0 0 0" rpy="0 0 0"/>
-        <mass value="${mass}"/>
+        <mass value="${wheel_mass}"/>
         <!-- Fórmula de inércia para cilindro sólido -->
         <inertia
-          ixx="${(1/12) * mass * (3*radius*radius + length*length)}"
+          ixx="${(1/12) * wheel_mass * (3*wheel_radius*wheel_radius + wheel_length*wheel_length)}"
           ixy="0.0" ixz="0.0"
-          iyy="${(1/12) * mass * (3*radius*radius + length*length)}"
+          iyy="${(1/12) * wheel_mass * (3*wheel_radius*wheel_radius + wheel_length*wheel_length)}"
           iyz="0.0"
-          izz="${(1/2) * mass * radius * radius}"/>
+          izz="${(1/2) * wheel_mass * wheel_radius * wheel_radius}"/>
       </inertial>
     </link>

Commit message: aps 1 feita

File: src/rm_description/urdf/differential_robot.xacro (robot description, xacro)
@@ -14,4 +14,7 @@
   <xacro:include filename="$(find rm_description)/urdf/properties.xacro"/>
   <xacro:include filename="$(find rm_description)/urdf/wheels.xacro"/>
+  <xacro:include filename="$(find rm_description)/urdf/gazebo_control.xacro"/>
+  <xacro:include filename="$(find rm_description)/urdf/sensors.xacro" />
+  <xacro:include filename="$(find rm_description)/urdf/inertial_macros.xacro"/>
   <!-- ==================== -->
   <!-- BASE FOOTPRINT       -->
@@ -50,14 +53,11 @@
       </geometry>
     </collision>
-    <inertial>
-      <origin xyz="0 0 0" rpy="0 0 0"/>
-      <mass value="${base_mass}"/>
-      <inertia
-        ixx="${(1/12) * base_mass * (3*base_width*base_width + base_height*base_height)}"
-        ixy="0.0" ixz="0.0"
-        iyy="${(1/12) * base_mass * (3*base_length*base_length + base_height*base_height)}"
-        iyz="0.0"
-        izz="${(1/2) * base_mass * base_length * base_length}"/>
-    </inertial>
+    <xacro:inertial_box
+        mass="${base_mass}"
+        x="${base_length}"
+        y="${base_width}"
+        z="${base_height}">
+      <origin xyz="0 0 0"/>
+    </xacro:inertial_box>
   </link>
   <joint name="base_joint" type="fixed">
@@ -90,11 +90,102 @@
   name="caster_ball"
   radius="0.1"
-  mass="0.7"
+  mass="1"
   material="red"/>
   <joint name="caster_joint" type="fixed">
   <parent link="base_link"/>
   <child link="caster_ball"/>
-  <origin xyz="0.25 0 -0.05"
+  <origin xyz="0.27 0 -0.05"
           rpy="0 0 0"/>
 </joint>
+<!-- ==================== -->
+<!-- CAMERA LINK -->
+<!-- ==================== -->
+<link name="camera">
+  <visual>
+    <origin xyz="0 0 0" rpy="0 0 0"/>
+    <geometry>
+      <box size="0.05 0.05 0.05"/>
+    </geometry>
+    <material name="green"/>
+  </visual>
+  <collision>
+    <origin xyz="0 0 0" rpy="0 0 0"/>
+    <geometry>
+      <box size="0.05 0.05 0.05"/>
+    </geometry>
+  </collision>
+  <inertial>
+    <origin xyz="0 0 0"/>
+    <mass value="0.1"/>
+    <inertia
+      ixx="0.0001"
+      ixy="0.0"
+      ixz="0.0"
+      iyy="0.0001"
+      iyz="0.0"
+      izz="0.0001"/>
+  </inertial>
+</link>
+<!-- ==================== -->
+<!-- CAMERA JOINT -->
+<!-- ==================== -->
+<joint name="camera_joint" type="fixed">
+  <parent link="base_link"/>
+  <child link="camera"/>
+  <!-- frente do robô -->
+  <origin xyz="-0.15 0 0" rpy="0 0 3.14159"/>
+</joint>
+<!-- ==================== -->
+<!-- IMU LINK -->
+<!-- ==================== -->
+<link name="IMU">
+</link>
+<!-- ==================== -->
+<!-- IMU JOINT -->
+<!-- ==================== -->
+<joint name="imu_joint" type="fixed">
+  <parent link="base_link"/>
+  <child link="IMU"/>
+  <!-- frente do robô -->
+  <origin xyz="0 0 0" rpy="0 0 0"/>
+</joint>
+<!-- ==================== -->
+<!-- LIDAR LINK -->
+<!-- ==================== -->
+<link name="lidar">
+  <visual>
+    <origin xyz="0 0 0" rpy="0 0 0"/>
+    <geometry>
+      <!-- cilindro achatado -->
+      <cylinder radius="0.06" length="0.02"/>
+    </geometry>
+    <material name="red"/>
+  </visual>
+  <collision>
+    <origin xyz="0 0 0" rpy="0 0 0"/>
+    <geometry>
+      <cylinder radius="0.06" length="0.02"/>
+    </geometry>
+  </collision>
+  <inertial>
+    <origin xyz="0 0 0"/>
+    <mass value="0.1"/>
+    <inertia
+      ixx="0.0001"
+      ixy="0"
+      ixz="0"
+      iyy="0.0001"
+      iyz="0"
+      izz="0.0001"/>
+  </inertial>
+</link>
+<!-- ==================== -->
+<!-- LIDAR JOINT -->
+<!-- ==================== -->
+<joint name="lidar_joint" type="fixed">
+  <parent link="base_link"/>
+  <child link="lidar"/>
+  <!-- em cima do robô -->
+  <origin xyz="0 0 ${base_height/2 + 0.06}" rpy="0 0 0"/>
+</joint>
 </robot>

File: src/rm_description/urdf/wheels.xacro (robot description, xacro)
@@ -1,4 +1,5 @@
 <?xml version="1.0"?>
 <robot xmlns:xacro="http://www.ros.org/wiki/xacro">
+  <xacro:include filename="$(find rm_description)/urdf/inertial_macros.xacro"/>
   <!-- ============================================ -->
   <!-- ARQUIVO DE MACROS                            -->
@@ -37,15 +38,10 @@
         </geometry>
       </collision>
-      <inertial>
-        <origin xyz="0 0 0" rpy="0 0 0"/>
-        <mass value="${wheel_mass}"/>
-        <!-- Fórmula de inércia para cilindro sólido -->
-        <inertia
-          ixx="${(1/12) * wheel_mass * (3*wheel_radius*wheel_radius + wheel_length*wheel_length)}"
-          ixy="0.0" ixz="0.0"
-          iyy="${(1/12) * wheel_mass * (3*wheel_radius*wheel_radius + wheel_length*wheel_length)}"
-          iyz="0.0"
-          izz="${(1/2) * wheel_mass * wheel_radius * wheel_radius}"/>
-      </inertial>
+      <xacro:inertial_cylinder
+        mass="${wheel_mass}"
+        length="${wheel_length}"
+        radius="${wheel_radius}">
+      <origin xyz="0 0 0"/>
+    </xacro:inertial_cylinder>
     </link>
   </xacro:macro>
@@ -76,15 +72,9 @@
         </geometry>
       </collision>
-      <inertial>
-        <origin xyz="0 0 0" rpy="0 0 0"/>
-        <mass value="${mass}"/>
-        <!-- Fórmula de inércia para esfera sólida -->
-        <inertia
-          ixx="${(2/5) * mass * radius * radius}"
-          ixy="0.0" ixz="0.0"
-          iyy="${(2/5) * mass * radius * radius}"
-          iyz="0.0"
-          izz="${(2/5) * mass * radius * radius}"/>
-      </inertial>
+      <xacro:inertial_sphere
+        mass="${mass}"
+        radius="${radius}">
+        <origin xyz="0 0 0"/>
+      </xacro:inertial_sphere>
     </link>
   </xacro:macro>
